File: pipistrelle.kicad_pcb (KiCad board)
At the start: 2 copper layers, 211.2 x 85.2 mm, 30 parts, among them SW10 SW_Push, SW11 SW_Push, SW12 SW_Push, SW14 SW_Push, SW15 SW_Push, SW16 SW_Push, SW17 SW_Push, SW18 SW_Push, SW2 SW_Push, SW20 SW_Push, SW21 SW_Push, SW22 SW_Push, SW23 SW_Push, SW24 SW_Push, SW25 SW_Push, SW26 SW_Push, SW3 SW_Push, SW4 SW_Push, SW5 SW_Push, SW6 SW_Push, SW8 SW_Push, SW9 SW_Push, U1 ProMicro-kbd

Commit message: Add files via upload
Parts:
- moved SW2 0.21 mm to (225.0, 98.8)
- moved SW17 0.11 mm to (205.7, 83.5)
- moved SW12 0.08 mm to (223.6, 81.9)

Commit message: Add files via upload
Parts:
- added SW18: SW_Push, Kailh:SW_PG1350_nonrev_DPB2, F.Cu at (105.0, 138.2)
- moved SW25 33.7 mm to (86.2, 139.0), turned to 5 degrees
- moved SW26 33.6 mm to (67.5, 141.4), turned to 10 degrees
- moved SW23 15.3 mm to (142.3, 141.4), turned to 350 degrees
- moved SW24 14.9 mm to (123.8, 139.1), turned to 355 degrees
Routing:
- net Switch18: track 0.00 -> 85.6 mm
- net Switch23: track 64.0 -> 82.1 mm
- net Switch20: track 70.7 -> 57.2 mm
- net Switch22: track 52.5 -> 64.8 mm
- net Switch21: track 53.6 -> 50.4 mm
Other:
- board size 211.2 x 85.2 mm -> 211.2 x 89.7 mm

Commit message: Add files via upload
Parts:
- added SW18: SW_Push, Kailh:SW_PG1350_nonrev_DPB2, F.Cu at (133.7, 138.4)
- moved SW24 28.7 mm to (152.5, 139.3)
- moved SW23 28.7 mm to (171.0, 141.8)
Routing:
- net Switch18: track 85.6 -> 114.7 mm
- net Switch20: track 57.2 -> 77.5 mm
- net Switch21: track 50.4 -> 61.2 mm

Commit message: new attenpt
Parts:
- removed Bat+1, BatGND1: MountingHole_Pad, kbd:1pin_conn
- removed RSW1: SW_Push, kbd:ResetSW
- removed the SW18 at (105.0, 138.2)
- removed SW_POWER1: SW_SPDT, Kailh:SPDT_C128955
- G***: moved to F.Cu
- moved SW4 152.3 mm to (223.0, 94.0), turned to 0 degrees
- moved SW2 148.3 mm to (79.0, 73.0), turned to 0 degrees
- moved SW3 116.1 mm to (169.0, 89.0), turned to 0 degrees
- moved SW5 98.1 mm to (187.0, 90.0), turned to 0 degrees
- moved U1 87.1 mm to (42.2, 81.9)
- moved SW18 80.6 mm to (97.0, 72.0), turned to 0 degrees
- moved SW20 79.5 mm to (115.0, 73.0), turned to 0 degrees
- moved SW26 32.4 mm to (97.0, 128.0), turned to 0 degrees
- moved SW25 32.0 mm to (115.0, 125.0), turned to 0 degrees
- moved SW6 31.0 mm to (133.0, 91.0), turned to 0 degrees
- moved SW8 30.7 mm to (115.0, 90.0), turned to 0 degrees
- moved SW9 30.4 mm to (97.0, 89.0), turned to 0 degrees
- moved SW6 29.7 mm to (133.0, 74.0), turned to 0 degrees
- moved SW10 29.4 mm to (79.0, 90.0), turned to 0 degrees
- moved SW11 27.9 mm to (61.0, 94.0), turned to 0 degrees
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Routing:
- net Switch3: track 58.0 -> 213.5 mm
- net Switch4: track 40.4 -> 180.9 mm
- net Switch11: track 46.6 -> 129.7 mm
- net Switch14: track 76.9 -> 160.0 mm
- net Switch19: track 27.8 -> 109.7 mm
- net Switch12: track 24.1 -> 105.8 mm
- net Switch17: track 83.8 -> 164.7 mm
- net Switch2: track 76.1 -> 157.0 mm
- net Switch13: track 61.3 -> 140.9 mm
- net Switch9: track 126.8 -> 49.0 mm
- net Switch20: track 77.5 -> 153.1 mm
- net Switch21: track 61.2 -> 135.8 mm
- net Switch5: track 65.6 -> 138.4 mm
- net Switch10: track 127.3 -> 198.2 mm
- net Switch6: track 44.5 -> 96.2 mm
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- added copper zone on B.Cu, net gnd
Other:
- board size 211.2 x 89.7 mm -> 200.6 x 82.5 mm
- board text added: "#"
- board text added: "*"

Commit message: small tidy
Routing:
- net Switch13: track 140.9 -> 144.1 mm
- net Switch14: track 160.0 -> 163.1 mm
- net Switch17: track 164.7 -> 165.9 mm
- net Switch19: track 109.7 -> 110.9 mm
- net Switch3: track 213.5 -> 214.7 mm
- net Switch6: track 96.2 -> 95.4 mm
- net Switch2: track 157.0 -> 157.6 mm

Commit message: Add files via upload
Parts:
- added RSW1: SW_PUSH, kbd:ResetSW_1side, F.Cu at (227.1, 65.6)
Routing:
- net reset: track 0.00 -> 246.5 mm
- net Switch2: track 157.6 -> 156.7 mm
- net Switch4: track 180.5 -> 179.5 mm
- net Switch5: track 138.0 -> 137.1 mm
- net Switch6: track 95.4 -> 94.5 mm
- net Switch10: track 198.2 -> 199.0 mm
- net Switch14: track 163.1 -> 164.0 mm
Other:
- outline, holes or cut-outs redrawn
